File: cv_lighting_pcb/cv_lighting_pcb.kicad_sch (KiCad schematic)
At the start: 24 parts, among them Q1 2N3906, U3 VO615A-9

Commit message: formatting changes
Parts:
- renumbered +32V to +32V1
Other:
- company: (none) -> UIUC Pacbot Team
- title: (none) -> Computer Vision Lighting Board
Changed lines of the file:
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@@
 (kicad_sch (version 20230121) (generator eeschema)
   (paper "A4")
+  (title_block
+    (title "Computer Vision Lighting Board")
+    (date "2023-11-21")
+    (rev "v.3.0")
+    (company "UIUC Pacbot Team")
+  )
   (junction (at 177.8 96.52) (diameter 0) (color 0 0 0 0)
   )
@@
   )
   (text "Control dimming: optocoupler or something\nSo far this circuit has 8 leds and one current driver"
-    (at 90.17 85.09 0)
+    (at 88.9 147.32 0)
     (effects (font (size 1.27 1.27)) (justify left bottom))
   )
@@
   (symbol (lib_id "cv_lighting_symbols:+32V") (at 86.36 99.06 90) (unit 1)
     (in_bom yes) (on_board yes) (dnp no)
-    (property "Reference" "+32V" (at 83.82 99.06 90)
+    (property "Reference" "+32V1" (at 83.82 99.06 90)
       (effects (font (size 1.27 1.27)) (justify right))
     )
@@
       (project "cv_lighting_pcb"
         (path "/d003750a-5843-4e2f-8a13-c4462072ff66"
-          (reference "+32V") (unit 1)
-        )
-      )
+          (reference "+32V1") (unit 1)
+        )
+      )
