File: cv_lighting_pcb/_autosave-cv_lighting_pcb.kicad_sch (KiCad schematic)
At the start: 24 parts, among them Q2 2N3904, U1 Current Driver, U2 Camera Input, U4 Barrel Jack

Commit message: more changes to cv lighting
Parts:
- Q2: value 2N3904 -> MMBT3904; footprint Package_TO_SOT_THT:TO-92_Inline -> cv_lighting_footprints:MMBT3904
Changed lines of the file:
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@@
       (effects (font (size 1.27 1.27)))
     )
-    (property "Value" "2N3904" (at 106.68 124.46 90)
+    (property "Value" "MMBT3904" (at 106.68 124.46 90)
       (effects (font (size 1.27 1.27)))
     )
-    (property "Footprint" "Package_TO_SOT_THT:TO-92_Inline" (at 104.775 125.73 0)
+    (property "Footprint" "cv_lighting_footprints:MMBT3904" (at 104.775 125.73 0)
       (effects (font (size 1.27 1.27) italic) (justify left) hide)
     )
