File: cv_lighting_pcb/cv_lighting_pcb.kicad_pcb (KiCad board)
At the start: 2 copper layers, 83.8 x 68.6 mm, 24 parts, among them Q2 MMBT3904, U1 Current Driver, U2 Camera Input, U4 Barrel Jack

Commit message: cv lighting final?
Parts:
- moved RV1 26.8 mm to (123.2, 82.8), turned to 90 degrees
- moved Q2 26.2 mm to (117.4, 77.8)
- moved R1 20.6 mm to (124.5, 86.4), turned to 180 degrees
- moved U2 19.1 mm to (124.2, 91.4), turned to -90 degrees
- moved U4 7.95 mm to (107.4, 92.3)
- moved C1 7.95 mm to (106.2, 82.0)
Routing:
- net Net-(Q2-E): track 79.1 -> 32.7 mm
- net Net-(Q2-C): track 73.6 -> 37.9 mm
- net Net-(D15-A): track 87.6 -> 75.4 mm
- net +30V: track 19.0 -> 22.7 mm
Other:
- board size 83.8 x 68.6 mm -> 83.8 x 61 mm

Commit message: [Generated Gerber Files and Drill Files]
Other:
- board text added: "GND"
Changed lines of the file:
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@@
 (kicad_pcb (version 20221018) (generator pcbnew)
   (general
-    (thickness 1.36532)
+    (thickness 1.35532)
   )
   (paper "A4")
@@
       (layer "dielectric 1" (type "prepreg") (color "FR4 natural") (thickness 0.1) (material "FR4") (epsilon_r 4.5) (loss_tangent 0.02))
       (layer "B.Cu" (type "copper") (thickness 1.2))
-      (layer "B.Mask" (type "Bottom Solder Mask") (thickness 0.01))
       (copper_finish "None")
       (dielectric_constraints no)
@@
     (pad_to_mask_clearance 0)
     (pcbplotparams
-      (layerselection 0x00010fc_7fffffff)
+      (layerselection 0x00010a8_7fffffff)
       (plot_on_all_layers_selection 0x0000000_00000000)
       (disableapertmacros false)
-      (usegerberextensions false)
+      (usegerberextensions true)
       (usegerberattributes true)
       (usegerberadvancedattributes true)
-      (creategerberjobfile true)
+      (creategerberjobfile false)
       (dashed_line_dash_ratio 12.000000)
       (dashed_line_gap_ratio 3.000000)
@@
       (plotinvisibletext false)
       (sketchpadsonfab false)
-      (subtractmaskfromsilk false)
+      (subtractmaskfromsilk true)
       (outputformat 1)
       (mirror false)
       (drillshape 0)
       (scaleselection 1)
-      (outputdirectory "")
+      (outputdirectory "Gerber/")
     )
   )
@@
         (effects (font (size 1 1) (thickness 0.15)))
     )
-    (fp_text value "Barrel Jack" (at -0.3556 -8.7884 90) (layer "F.Fab")
+    (fp_text value "Barrel Jack" (at -0.3556 -8.7884 90) (layer "F.SilkS")
         (effects (font (size 1 1) (thickness 0.15)))
     )
@@
   (gr_line (start 156.5 82) (end 170.7 67.8)
     (stroke (width 0.1) (type default)) (layer "F.Fab"))
+  (gr_text "hole for wire \nfrom camera to pcb\n\n" (at 111.76 111.76) (layer "F.SilkS")
+    (effects (font (size 1 1) (thickness 0.125)) (justify left bottom))
+  )
   (gr_text "UIUC Pacbot 2023-24\nCV Lighting PCB\nDesigned by Ansley, Tim, Jake" (at 129.54 109.22) (layer "F.SilkS")
     (effects (font (size 1 1) (thickness 0.15)) (justify left bottom))
   )
-  (gr_text "hole for wire from camera to pcb\n\n" (at 116.84 104.14) (layer "F.Fab")
+  (gr_text "GND" (at 104.14 101.6) (layer "F.SilkS")
     (effects (font (size 1 1) (thickness 0.15)) (justify left bottom))
   )
