File: pacboard2025_alt/pacboard2025_alt.kicad_sch (KiCad schematic)
At the start: 31 parts, among them J1 XT30 Male Connector, Q1 NMOS, U2 D24V50F5, U3 ProS3

Commit message: schematic from 10/19
Parts:
- added C6: 100n, symbol Device:C
- added R10: 200, symbol Device:R_US
- added R7, R8, R9: 10k, symbol Device:R_US
- added U1: INA237AQDGSRQ1, U_VSSOP10_DGS_TEX, symbol pacbotsym:INA237AQDGSRQ1
Connections:
- net GND is gone; now on net BAT_12V: C1.2, C2.2, C3.2, C4.2, C5.2, J1.1 (Pin_1), LED1.1 (GND), LED2.1 (GND), LED3.1 (GND), LED4.1 (GND), LP3470A1.2 (GND), MC1.13 (GND), MC1.2 (GND), MC1.5 (PMODE), MC2.13 (GND), MC2.2 (GND), MC2.5 (PMODE), MOTOR1.5 (Pin_5), MOTOR2.5 (Pin_5), Q1.2 (S), R1.2, R5.2, R6.2, STEMMA_QT1.1 (Pin_1), U2.2 (GND), U2.3 (GND), U3.2 (GND), U3.25 (GND)
- net 5V: now also C6.1, R7.1, R8.1, R9.1, U1.6 (VS)
- net BAT_12V: now also C6.2, R10.1, U1.1 (A1), U1.10 (IN+), U1.2 (A0), U1.7 (GND), U1.8 (VBUS)
- net SERIAL_CLOCK_LINE: now also R7.2, U1.5 (SCL)
- net SERIAL_DATA_LINE: now also R8.2, U1.4 (SDA)
- new net: R9.2, U1.3 (ALERT)
- new net 12V_After: R10.2, U1.9 (IN-)
