File: pacboard_2026/pacboard_2026.kicad_sch (KiCad schematic)
At the start: 13 parts, among them J1 STEMMA_QT1, J2 STEMMA_QT2, J3 STEMMA_QT3, J4 STEMMA_QT4, J5 STEMMA_QT5, J6 STEMMA_QT6, J7 Conn_01x02, M1 Conn_01x06_Pin, M2 Conn_01x06_Pin, U1 Arduino Nano ESP32, U2 DRV8876, U3 DRV8876

Commit message: Add files via upload
Parts:
- added C1: 0.1uF, Capacitor_SMD:C_0805_2012Metric_Pad1.18x1.45mm_HandSolder, symbol Device:C
- added R1, R3: 10k, Resistor_SMD:R_0805_2012Metric_Pad1.20x1.40mm_HandSolder, symbol Device:R_US
- added R2: 15k, Resistor_SMD:R_0805_2012Metric_Pad1.20x1.40mm_HandSolder, symbol Device:R_US
- added U4: LP3470A1, Package_TO_SOT_SMD:SOT-23-5, symbol pacboard_custom:LP3470A1
- added U5: NMOS, board1_footprints:IFX-PG-TSDSON-8-901-G-V, symbol pacboard_custom:pacboard_nmos
Connections:
- net 12V: now also U5.1 (S), U5.2 (S), U5.3 (S)
- net BAT_12V: now also C1.2, R1.1, R2.1, U5.5 (D), U5.6 (D), U5.7 (D), U5.8 (D)
- net GND: now also C1.1, R3.2, U4.2 (GND)
- new net: R2.2, R3.1, U4.3 (VCC1), U4.4 (VCC)
- new net: R1.2, U4.5 (~RST), U5.4 (G)
- no-connect marks 19 -> 22
